Commit message: feat: Enhance error handling and diagnostics in SoArmMoce
- Improved error payload structure to include additional details from exceptions.
- Added a new script for read-only IK diagnostics, allowing users to diagnose inverse kinematics without moving hardware.
- Extended the movement commands in the SoArmMoceController to support tracing of joint movements, capturing detailed state information during execution.
- Introduced multi-turn joint handling to accurately track joint positions across multiple revolutions.
- Implemented a model diagnosis feature that provides kinematic reports based on current joint states and offset hypotheses.
- Enhanced the state reading functionality to include detailed reports on joint positions and calibration data.

File: sdk/src/soarmmoce_sdk/resources/urdf/soarmoce_urdf.urdf (robot description, URDF)
Before this commit: robot soarmoce_urdf, 7 links, 6 joints
Joints:
- joint wrist: limit lower=-1.30000000 upper=1.30000000 effort=0 velocity=0 -> lower=-1.30000000 upper=1.31000000 effort=0 velocity=0
